File: kicad/pico_tcs.kicad_sch (KiCad schematic)
At the start: 14 parts, among them J1 TCS In, J2 Conn_01x20_Male, J3 Conn_01x20_Male, J4 Keypad, J5 Display, U1 L7805, U2 ULN2003

Commit message: Dateien hochladen nach „kicad“
Connections:
- net at J3.7 (Pin_7): now also R3.1, R4.2
- net at J2.1 (Pin_1): no longer R5.1
- net at J2.20 (Pin_20): now also R5.1
- now unconnected: J2.2 (Pin_2)
Changed lines of the file:
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@@
-    (stroke (width 0) (type default) (color 0 0 0 0))
-  )
-  (wire (pts (xy 107.95 39.37) (xy 128.27 39.37))
     (stroke (width 0) (type default) (color 0 0 0 0))
   )
@@
     (stroke (width 0) (type default) (color 0 0 0 0))
   )
-  (wire (pts (xy 99.06 25.4) (xy 99.06 41.91))
-    (stroke (width 0) (type default) (color 0 0 0 0))
-  )
   (wire (pts (xy 71.12 54.61) (xy 71.12 60.96))
     (stroke (width 0) (type default) (color 0 0 0 0))
   )
   (wire (pts (xy 119.38 62.23) (xy 128.27 62.23))
+    (stroke (width 0) (type default) (color 0 0 0 0))
+  )
+  (wire (pts (xy 148.59 25.4) (xy 148.59 54.61))
     (stroke (width 0) (type default) (color 0 0 0 0))
   )
@@
     (stroke (width 0) (type default) (color 0 0 0 0))
   )
-  (wire (pts (xy 86.36 25.4) (xy 99.06 25.4))
+  (wire (pts (xy 107.95 87.63) (xy 128.27 87.63))
     (stroke (width 0) (type default) (color 0 0 0 0))
   )
@@
   )
   (wire (pts (xy 119.38 77.47) (xy 128.27 77.47))
-    (stroke (width 0) (type default) (color 0 0 0 0))
-  )
-  (wire (pts (xy 107.95 20.32) (xy 107.95 39.37))
     (stroke (width 0) (type default) (color 0 0 0 0))
   )
@@
     (stroke (width 0) (type default) (color 0 0 0 0))
   )
-  (wire (pts (xy 99.06 41.91) (xy 128.27 41.91))
-    (stroke (width 0) (type default) (color 0 0 0 0))
-  )
   (wire (pts (xy 119.38 64.77) (xy 128.27 64.77))
     (stroke (width 0) (type default) (color 0 0 0 0))
@@
   )
   (wire (pts (xy 86.36 41.91) (xy 88.9 41.91))
+    (stroke (width 0) (type default) (color 0 0 0 0))
+  )
+  (wire (pts (xy 107.95 20.32) (xy 107.95 87.63))
     (stroke (width 0) (type default) (color 0 0 0 0))
   )
@@
   )
   (wire (pts (xy 64.77 33.02) (xy 64.77 41.91))
+    (stroke (width 0) (type default) (color 0 0 0 0))
+  )
+  (wire (pts (xy 148.59 54.61) (xy 140.97 54.61))
     (stroke (width 0) (type default) (color 0 0 0 0))
   )
@@
     (stroke (width 0) (type default) (color 0 0 0 0))
   )
+  (wire (pts (xy 86.36 25.4) (xy 148.59 25.4))
+    (stroke (width 0) (type default) (color 0 0 0 0))
+  )
