File: kicad/power_from_tcs_bus/pico_tcs.kicad_pcb (KiCad board)
At the start: 2 copper layers, 90.2 x 65.3 mm, 14 parts, among them J1 TCS In, J2 Conn_01x20_Male, J3 Conn_01x20_Male, J4 Keypad, J5 Display, U1 L7805, U2 ULN2003

Commit message: Dateien hochladen nach „kicad/power_from_tcs_bus“
fixed bug in connection between display and pico
Connections:
- J2 pad 10: Net-(J2-Pad10) -> Net-(J5-Pad4)
- J2 pad 11: Net-(J2-Pad11) -> Net-(J5-Pad5)
- J2 pad 12: Net-(J2-Pad12) -> Net-(J5-Pad6)
- J2 pad 13: Net-(J2-Pad13) -> unconnected-(J2-Pad13)
- J2 pad 9: unconnected-(J2-Pad9) -> Net-(J5-Pad3)
- J5 pad 3: Net-(J2-Pad10) -> Net-(J5-Pad3)
- J5 pad 4: Net-(J2-Pad11) -> Net-(J5-Pad4)
- J5 pad 5: Net-(J2-Pad12) -> Net-(J5-Pad5)
- J5 pad 6: Net-(J2-Pad13) -> Net-(J5-Pad6)
Routing:
- net Net-(J5-Pad6): track 0.00 -> 7.97 mm
- net Net-(J5-Pad5): track 0.00 -> 7.97 mm
- net Net-(J5-Pad4): track 0.00 -> 7.97 mm
- net Net-(J5-Pad3): track 0.00 -> 7.92 mm
- net Net-(J2-Pad12): track 6.90 -> 0.00 mm
- net Net-(J2-Pad11): track 6.90 -> 0.00 mm
- net Net-(J2-Pad10): track 6.90 -> 0.00 mm
- net Net-(J2-Pad13): track 6.90 -> 0.00 mm
Other:
- board text added: "v1.3 © by Manuel Kamper 03.01.2023"
- board text removed: "v1.0 © by Manuel Kamper 17.12.2022"
Changed lines of the file:
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@@
   (net 8 "unconnected-(J2-Pad7)")
   (net 9 "unconnected-(J2-Pad8)")
-  (net 10 "unconnected-(J2-Pad9)")
+  (net 10 "Net-(J5-Pad3)")
   (net 11 "unconnected-(J2-Pad17)")
   (net 12 "unconnected-(J2-Pad18)")
@@
   (net 29 "Net-(J3-Pad16)")
   (net 30 "Net-(J3-Pad17)")
-  (net 31 "Net-(J2-Pad10)")
-  (net 32 "Net-(J2-Pad11)")
-  (net 33 "Net-(J2-Pad12)")
-  (net 34 "Net-(J2-Pad13)")
-  (net 35 "Net-(J2-Pad14)")
-  (net 36 "Net-(J2-Pad15)")
-  (net 37 "Net-(J2-Pad16)")
+  (net 31 "Net-(J5-Pad4)")
+  (net 32 "Net-(J5-Pad5)")
+  (net 33 "Net-(J5-Pad6)")
+  (net 34 "unconnected-(J2-Pad13)")
+  (net 35 "Net-(J5-Pad7)")
+  (net 36 "Net-(J5-Pad8)")
+  (net 37 "Net-(J5-Pad9)")
   (net 38 "Net-(J3-Pad2)")
   (net 39 "unconnected-(U2-Pad2)")
@@
   (net 52 "unconnected-(J2-Pad1)")
   (net 53 "unconnected-(J2-Pad2)")
-  (net 54 "Net-(R3-Pad1)")
+  (net 54 "Net-(J3-Pad7)")
   (net 55 "Net-(R1-Pad1)")
   (net 56 "Net-(R5-Pad2)")
@@
       (net 2 "GND") (pintype "passive"))
     (pad "2" thru_hole oval (at 10.16 0 180) (size 1.6 1.6) (drill 0.8) (layers *.Cu *.Mask)
-      (net 54 "Net-(R3-Pad1)") (pintype "passive"))
+      (net 54 "Net-(J3-Pad7)") (pintype "passive"))
     (model "${KICAD6_3DMODEL_DIR}/Resistor_THT.3dshapes/R_Axial_DIN0207_L6.3mm_D2.5mm_P10.16mm_Horizontal.wrl"
       (offset (xyz 0 0 0))
@@
       (net 16 "unconnected-(J3-Pad6)") (pinfunction "Pin_6") (pintype "passive"))
     (pad "7" thru_hole oval (at 0 15.24) (size 1.7 1.7) (drill 1) (layers *.Cu *.Mask)
-      (net 54 "Net-(R3-Pad1)") (pinfunction "Pin_7") (pintype "passive"))
+      (net 54 "Net-(J3-Pad7)") (pinfunction "Pin_7") (pintype "passive"))
     (pad "8" thru_hole oval (at 0 17.78) (size 1.7 1.7) (drill 1) (layers *.Cu *.Mask)
       (net 18 "unconnected-(J3-Pad8)") (pinfunction "Pin_8") (pintype "passive"))
@@
       (net 9 "unconnected-(J2-Pad8)") (pinfunction "Pin_8") (pintype "passive"))
     (pad "9" thru_hole oval (at 0 20.32) (size 1.7 1.7) (drill 1) (layers *.Cu *.Mask)
-      (net 10 "unconnected-(J2-Pad9)") (pinfunction "Pin_9") (pintype "passive"))
+      (net 10 "Net-(J5-Pad3)") (pinfunction "Pin_9") (pintype "passive"))
     (pad "10" thru_hole oval (at 0 22.86) (size 1.7 1.7) (drill 1) (layers *.Cu *.Mask)
-      (net 31 "Net-(J2-Pad10)") (pinfunction "Pin_10") (pintype "passive"))
+      (net 31 "Net-(J5-Pad4)") (pinfunction "Pin_10") (pintype "passive"))
     (pad "11" thru_hole oval (at 0 25.4) (size 1.7 1.7) (drill 1) (layers *.Cu *.Mask)
-      (net 32 "Net-(J2-Pad11)") (pinfunction "Pin_11") (pintype "passive"))
+      (net 32 "Net-(J5-Pad5)") (pinfunction "Pin_11") (pintype "passive"))
     (pad "12" thru_hole oval (at 0 27.94) (size 1.7 1.7) (drill 1) (layers *.Cu *.Mask)
-      (net 33 "Net-(J2-Pad12)") (pinfunction "Pin_12") (pintype "passive"))
+      (net 33 "Net-(J5-Pad6)") (pinfunction "Pin_12") (pintype "passive"))
     (pad "13" thru_hole oval (at 0 30.48) (size 1.7 1.7) (drill 1) (layers *.Cu *.Mask)
-      (net 34 "Net-(J2-Pad13)") (pinfunction "Pin_13") (pintype "passive"))
+      (net 34 "unconnected-(J2-Pad13)") (pinfunction "Pin_13") (pintype "passive"))
     (pad "14" thru_hole oval (at 0 33.02) (size 1.7 1.7) (drill 1) (layers *.Cu *.Mask)
-      (net 35 "Net-(J2-Pad14)") (pinfunction "Pin_14") (pintype "passive"))
+      (net 35 "Net-(J5-Pad7)") (pinfunction "Pin_14") (pintype "passive"))
     (pad "15" thru_hole oval (at 0 35.56) (size 1.7 1.7) (drill 1) (layers *.Cu *.Mask)
-      (net 36 "Net-(J2-Pad15)") (pinfunction "Pin_15") (pintype "passive"))
+      (net 36 "Net-(J5-Pad8)") (pinfunction "Pin_15") (pintype "passive"))
     (pad "16" thru_hole oval (at 0 38.1) (size 1.7 1.7) (drill 1) (layers *.Cu *.Mask)
-      (net 37 "Net-(J2-Pad16)") (pinfunction "Pin_16") (pintype "passive"))
+      (net 37 "Net-(J5-Pad9)") (pinfunction "Pin_16") (pintype "passive"))
     (pad "17" thru_hole oval (at 0 40.64) (size 1.7 1.7) (drill 1) (layers *.Cu *.Mask)
       (net 11 "unconnected-(J2-Pad17)") (pinfunction "Pin_17") (pintype "passive"))
@@
       (net 2 "GND") (pinfunction "Pin_2") (pintype "passive"))
     (pad "3" thru_hole oval (at 0 5.08) (size 1.7 1.7) (drill 1) (layers *.Cu *.Mask)
-      (net 31 "Net-(J2-Pad10)") (pinfunction "Pin_3") (pintype "passive"))
+      (net 10 "Net-(J5-Pad3)") (pinfunction "Pin_3") (pintype "passive"))
     (pad "4" thru_hole oval (at 0 7.62) (size 1.7 1.7) (drill 1) (layers *.Cu *.Mask)
-      (net 32 "Net-(J2-Pad11)") (pinfunction "Pin_4") (pintype "passive"))
+      (net 31 "Net-(J5-Pad4)") (pinfunction "Pin_4") (pintype "passive"))
     (pad "5" thru_hole oval (at 0 10.16) (size 1.7 1.7) (drill 1) (layers *.Cu *.Mask)
-      (net 33 "Net-(J2-Pad12)") (pinfunction "Pin_5") (pintype "passive"))
+      (net 32 "Net-(J5-Pad5)") (pinfunction "Pin_5") (pintype "passive"))
     (pad "6" thru_hole oval (at 0 12.7) (size 1.7 1.7) (drill 1) (layers *.Cu *.Mask)
-      (net 34 "Net-(J2-Pad13)") (pinfunction "Pin_6") (pintype "passive"))
+      (net 33 "Net-(J5-Pad6)") (pinfunction "Pin_6") (pintype "passive"))
     (pad "7" thru_hole oval (at 0 15.24) (size 1.7 1.7) (drill 1) (layers *.Cu *.Mask)
-      (net 35 "Net-(J2-Pad14)") (pinfunction "Pin_7") (pintype "passive"))
+      (net 35 "Net-(J5-Pad7)") (pinfunction "Pin_7") (pintype "passive"))
     (pad "8" thru_hole oval (at 0 17.78) (size 1.7 1.7) (drill 1) (layers *.Cu *.Mask)
-      (net 36 "Net-(J2-Pad15)") (pinfunction "Pin_8") (pintype "passive"))
+      (net 36 "Net-(J5-Pad8)") (pinfunction "Pin_8") (pintype "passive"))
     (pad "9" thru_hole oval (at 0 20.32) (size 1.7 1.7) (drill 1) (layers *.Cu *.Mask)
-      (net 37 "Net-(J2-Pad16)") (pinfunction "Pin_9") (pintype "passive"))
+      (net 37 "Net-(J5-Pad9)") (pinfunction "Pin_9") (pintype "passive"))
     (model "${KICAD6_3DMODEL_DIR}/Connector_PinSocket_2.54mm.3dshapes/PinSocket_1x09_P2.54mm_Vertical.wrl"
       (offset (xyz 0 0 0))
@@
     (fp_line (start 1.93 -1.25) (end 1.93 1.25) (layer "F.Fab") (width 0.1))
     (pad "1" thru_hole circle (at 0 0 270) (size 1.6 1.6) (drill 0.8) (layers *.Cu *.Mask)
-      (net 54 "Net-(R3-Pad1)") (pintype "passive"))
+      (net 54 "Net-(J3-Pad7)") (pintype "passive"))
     (pad "2" thru_hole oval (at 10.16 0 270) (size 1.6 1.6) (drill 0.8) (layers *.Cu *.Mask)
       (net 17 "Net-(J1-Pad1)") (pintype "passive"))
@@
     (effects (font (size 1.5 1.5) (thickness 0.3)))
   )
-  (gr_text "v1.0 © by Manuel Kamper 17.12.2022" (at 156.21 120.904) (layer "F.SilkS")
+  (gr_text "v1.3 © by Manuel Kamper 03.01.2023" (at 156.21 120.904) (layer "F.SilkS")
     (effects (font (size 1.5 1.5) (thickness 0.375)))
   )
@@
   (segment (start 193.982369 87.376) (end 193.982369 76.695369) (width 1.5) (layer "B.Cu") (net 3))
   (segment (start 191.657 74.37) (end 184.627 67.34) (width 1.5) (layer "B.Cu") (net 3))
+  (segment (start 142.295 90.17) (end 144.805 87.66) (width 1) (layer "B.Cu") (net 10))
+  (segment (start 137.922 90.17) (end 142.295 90.17) (width 1) (layer "B.Cu") (net 10))
   (segment (start 120.65 115.57) (end 114.3 109.22) (width 1) (layer "B.Cu") (net 17))
   (segment (start 120.65 115.57) (end 120.65 118.11) (width 1) (layer "B.Cu") (net 17))
@@
   (segment (start 169.926 107.95) (end 162.615 107.95) (width 1) (layer "B.Cu") (net 30))
   (segment (start 162.615 107.95) (end 162.585 107.98) (width 0.25) (layer "B.Cu") (net 30))
+  (segment (start 142.295 92.71) (end 144.805 90.2) (width 1) (layer "B.Cu") (net 31))
   (segment (start 144.775 90.17) (end 144.805 90.2) (width 0.25) (layer "B.Cu") (net 31))
-  (segment (start 137.922 90.17) (end 144.775 90.17) (width 1) (layer "B.Cu") (net 31))
-  (segment (start 137.922 92.71) (end 144.775 92.71) (width 1) (layer "B.Cu") (net 32))
+  (segment (start 137.922 92.71) (end 142.295 92.71) (width 1) (layer "B.Cu") (net 31))
+  (segment (start 137.922 95.25) (end 142.295 95.25) (width 1) (layer "B.Cu") (net 32))
+  (segment (start 142.295 95.25) (end 144.805 92.74) (width 1) (layer "B.Cu") (net 32))
   (segment (start 144.775 92.71) (end 144.805 92.74) (width 0.25) (layer "B.Cu") (net 32))
+  (segment (start 137.922 97.79) (end 142.295 97.79) (width 1) (layer "B.Cu") (net 33))
+  (segment (start 142.295 97.79) (end 144.805 95.28) (width 1) (layer "B.Cu") (net 33))
   (segment (start 144.775 95.25) (end 144.805 95.28) (width 0.25) (layer "B.Cu") (net 33))
-  (segment (start 137.922 95.25) (end 144.775 95.25) (width 1) (layer "B.Cu") (net 33))
   (segment (start 144.775 97.79) (end 144.805 97.82) (width 0.25) (layer "B.Cu") (net 34))
-  (segment (start 137.922 97.79) (end 144.775 97.79) (width 1) (layer "B.Cu") (net 34))
   (segment (start 137.922 100.33) (end 144.775 100.33) (width 1) (layer "B.Cu") (net 35))
   (segment (start 144.775 100.33) (end 144.805 100.36) (width 0.25) (layer "B.Cu") (net 35))
