File: kicad/power_via_9-24v_source/pico_tcs.kicad_pcb (KiCad board)
At the start: 2 copper layers, 90.2 x 65.3 mm, 14 parts, among them J1 TCS/Power, J2 Conn_01x20_Male, J3 Conn_01x20_Male, J4 Keypad, J5 Display, U1 L7805, U2 ULN2003

Commit message: fixed bug in connection between display and pico
Connections:
- J2 pad 13: Net-(J2-Pad13) -> unconnected-(J2-Pad13)
- J2 pad 9: unconnected-(J2-Pad9) -> Net-(J2-Pad9)
- J5 pad 3: Net-(J2-Pad10) -> Net-(J2-Pad9)
- J5 pad 4: Net-(J2-Pad11) -> Net-(J2-Pad10)
- J5 pad 5: Net-(J2-Pad12) -> Net-(J2-Pad11)
- J5 pad 6: Net-(J2-Pad13) -> Net-(J2-Pad12)
Routing:
- net Net-(J2-Pad9): track 0.00 -> 7.92 mm
- net Net-(J2-Pad13): track 6.90 -> 0.00 mm
- net Net-(J2-Pad12): track 6.90 -> 7.97 mm
- net Net-(J2-Pad11): track 6.90 -> 7.97 mm
- net Net-(J2-Pad10): track 6.90 -> 7.97 mm
Other:
- board text added: "v1.5 © by Manuel Kamper 03.01.2023"
- board text removed: "v1.1 © by Manuel Kamper 19.12.2022"
Changed lines of the file:
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@@
   (net 8 "unconnected-(J2-Pad7)")
   (net 9 "unconnected-(J2-Pad8)")
-  (net 10 "unconnected-(J2-Pad9)")
+  (net 10 "Net-(J2-Pad9)")
   (net 11 "unconnected-(J2-Pad17)")
   (net 12 "unconnected-(J2-Pad18)")
@@
   (net 31 "Net-(J2-Pad11)")
   (net 32 "Net-(J2-Pad12)")
-  (net 33 "Net-(J2-Pad13)")
+  (net 33 "unconnected-(J2-Pad13)")
   (net 34 "Net-(J2-Pad14)")
   (net 35 "Net-(J2-Pad15)")
@@
       (net 9 "unconnected-(J2-Pad8)") (pinfunction "Pin_8") (pintype "passive"))
     (pad "9" thru_hole oval (at 0 20.32) (size 1.7 1.7) (drill 1) (layers *.Cu *.Mask)
-      (net 10 "unconnected-(J2-Pad9)") (pinfunction "Pin_9") (pintype "passive"))
+      (net 10 "Net-(J2-Pad9)") (pinfunction "Pin_9") (pintype "passive"))
     (pad "10" thru_hole oval (at 0 22.86) (size 1.7 1.7) (drill 1) (layers *.Cu *.Mask)
       (net 30 "Net-(J2-Pad10)") (pinfunction "Pin_10") (pintype "passive"))
@@
       (net 32 "Net-(J2-Pad12)") (pinfunction "Pin_12") (pintype "passive"))
     (pad "13" thru_hole oval (at 0 30.48) (size 1.7 1.7) (drill 1) (layers *.Cu *.Mask)
-      (net 33 "Net-(J2-Pad13)") (pinfunction "Pin_13") (pintype "passive"))
+      (net 33 "unconnected-(J2-Pad13)") (pinfunction "Pin_13") (pintype "passive"))
     (pad "14" thru_hole oval (at 0 33.02) (size 1.7 1.7) (drill 1) (layers *.Cu *.Mask)
       (net 34 "Net-(J2-Pad14)") (pinfunction "Pin_14") (pintype "passive"))
@@
       (net 2 "GND") (pinfunction "Pin_2") (pintype "passive"))
     (pad "3" thru_hole oval (at 0 5.08) (size 1.7 1.7) (drill 1) (layers *.Cu *.Mask)
-      (net 30 "Net-(J2-Pad10)") (pinfunction "Pin_3") (pintype "passive"))
+      (net 10 "Net-(J2-Pad9)") (pinfunction "Pin_3") (pintype "passive"))
     (pad "4" thru_hole oval (at 0 7.62) (size 1.7 1.7) (drill 1) (layers *.Cu *.Mask)
-      (net 31 "Net-(J2-Pad11)") (pinfunction "Pin_4") (pintype "passive"))
+      (net 30 "Net-(J2-Pad10)") (pinfunction "Pin_4") (pintype "passive"))
     (pad "5" thru_hole oval (at 0 10.16) (size 1.7 1.7) (drill 1) (layers *.Cu *.Mask)
-      (net 32 "Net-(J2-Pad12)") (pinfunction "Pin_5") (pintype "passive"))
+      (net 31 "Net-(J2-Pad11)") (pinfunction "Pin_5") (pintype "passive"))
     (pad "6" thru_hole oval (at 0 12.7) (size 1.7 1.7) (drill 1) (layers *.Cu *.Mask)
-      (net 33 "Net-(J2-Pad13)") (pinfunction "Pin_6") (pintype "passive"))
+      (net 32 "Net-(J2-Pad12)") (pinfunction "Pin_6") (pintype "passive"))
     (pad "7" thru_hole oval (at 0 15.24) (size 1.7 1.7) (drill 1) (layers *.Cu *.Mask)
       (net 34 "Net-(J2-Pad14)") (pinfunction "Pin_7") (pintype "passive"))
@@
     (effects (font (size 1.5 1.5) (thickness 0.3)))
   )
-  (gr_text "v1.1 © by Manuel Kamper 19.12.2022" (at 156.21 120.904) (layer "F.SilkS")
+  (gr_text "v1.5 © by Manuel Kamper 03.01.2023" (at 156.21 120.904) (layer "F.SilkS")
     (effects (font (size 1.5 1.5) (thickness 0.375)))
   )
@@
   (segment (start 184.627 67.34) (end 162.585 67.34) (width 1.5) (layer "B.Cu") (net 3))
   (segment (start 191.657 74.37) (end 184.627 67.34) (width 1.5) (layer "B.Cu") (net 3))
+  (segment (start 137.922 90.17) (end 142.295 90.17) (width 1) (layer "B.Cu") (net 10))
+  (segment (start 142.295 90.17) (end 144.805 87.66) (width 1) (layer "B.Cu") (net 10))
   (segment (start 162.615 97.79) (end 162.585 97.82) (width 0.25) (layer "B.Cu") (net 25))
   (segment (start 169.926 97.79) (end 162.615 97.79) (width 1) (layer "B.Cu") (net 25))
@@
   (segment (start 162.615 107.95) (end 162.585 107.98) (width 0.25) (layer "B.Cu") (net 29))
   (segment (start 144.775 90.17) (end 144.805 90.2) (width 0.25) (layer "B.Cu") (net 30))
-  (segment (start 137.922 90.17) (end 144.775 90.17) (width 1) (layer "B.Cu") (net 30))
-  (segment (start 137.922 92.71) (end 144.775 92.71) (width 1) (layer "B.Cu") (net 31))
+  (segment (start 137.922 92.71) (end 142.295 92.71) (width 1) (layer "B.Cu") (net 30))
+  (segment (start 142.295 92.71) (end 144.805 90.2) (width 1) (layer "B.Cu") (net 30))
+  (segment (start 137.922 95.25) (end 142.295 95.25) (width 1) (layer "B.Cu") (net 31))
   (segment (start 144.775 92.71) (end 144.805 92.74) (width 0.25) (layer "B.Cu") (net 31))
+  (segment (start 142.295 95.25) (end 144.805 92.74) (width 1) (layer "B.Cu") (net 31))
   (segment (start 144.775 95.25) (end 144.805 95.28) (width 0.25) (layer "B.Cu") (net 32))
-  (segment (start 137.922 95.25) (end 144.775 95.25) (width 1) (layer "B.Cu") (net 32))
+  (segment (start 142.295 97.79) (end 144.805 95.28) (width 1) (layer "B.Cu") (net 32))
+  (segment (start 137.922 97.79) (end 142.295 97.79) (width 1) (layer "B.Cu") (net 32))
   (segment (start 144.775 97.79) (end 144.805 97.82) (width 0.25) (layer "B.Cu") (net 33))
-  (segment (start 137.922 97.79) (end 144.775 97.79) (width 1) (layer "B.Cu") (net 33))
   (segment (start 137.922 100.33) (end 144.775 100.33) (width 1) (layer "B.Cu") (net 34))
   (segment (start 144.775 100.33) (end 144.805 100.36) (width 0.25) (layer "B.Cu") (net 34))
